File: eagle-cad/usb-pd.brd (EAGLE design)
At the start: 68.6 x 53.3 mm, 49 parts, among them Q1 CERAMIC_RESONATOR_SMD6M00G53Z, T1 FDN360P

Commit message: Went to a 4-layer board design with a stackup of signal, GND, VCC, signal
Parts:
- added D11: (no value), led:CHIPLED_0603
- added R16: 300, rcl:R0402
- moved C9 0.38 mm to (20.1, 32.9)
- moved R6 0.38 mm to (14.4, 41.7)
- moved U$3 0.25 mm to (11.8, 43.9), turned to 0 degrees
- moved R14 0.13 mm to (60.7, 20.5)
- moved R15 0.13 mm to (60.7, 19.3)
Connections:
- new net N$16: D11.A, R16.1
- net GND: now also D11.C
- net MOSI: now also R16.2
Routing:
- net +5V: track 214.6 -> 62.1 mm
- net VBUS: track 32.5 -> 18.5 mm, vias 3 -> 5
- net MISO: track 43.1 -> 39.0 mm, vias 2 -> 1
- net USB+: track 66.2 -> 70.3 mm
- net USB-: track 64.7 -> 68.4 mm
- net N$6: track 13.1 -> 9.50 mm
- net N$8: track 2.47 -> 5.61 mm, vias 0 -> 2
- net IO2: track 97.3 -> 95.0 mm
- net SCLK: track 37.6 -> 39.3 mm
- net GND: track 22.0 -> 20.4 mm, vias 75 -> 63
- net N$16: track 0.00 -> 1.52 mm
- net MOSI: track 34.5 -> 36.0 mm
- net N$5: track 6.44 -> 5.01 mm
- net PD_SCL: track 91.9 -> 90.7 mm
- net +3V3: track 64.8 -> 65.9 mm
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- added copper zone on layer 15, net +5V
- added copper zone on layer 2, net GND
- added copper zone on layer 15, net VBUS
