File: eagle-cad/usb-pd.sch (EAGLE design)
At the start: 49 parts, among them Q1 CERAMIC_RESONATOR_SMD6M00G53Z, T1 FDN360P

Commit message: Went to a 4-layer board design with a stackup of signal, GND, VCC, signal
Parts:
- added D11: (no value), led:LEDCHIPLED_0603
- added R16: 300, rcl:R-US_R0402
Connections:
- new net N$16: D11.A, R16.1
- net GND: now also D11.C
- net MOSI: now also R16.2
Changed lines of the file:
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@@
 <?xml version="1.0" encoding="utf-8"?>
 <!DOCTYPE eagle SYSTEM "eagle.dtd">
-<eagle version="7.7.0">
+<eagle version="7.6.0">
 <drawing>
 <settings>
@@
 <part name="T1" library="transistor-power" deviceset="FDN360P" device=""/>
 <part name="J$1" library="usb-pd" deviceset="TYPE-C-12401548E4" device=""/>
+<part name="R16" library="rcl" deviceset="R-US_" device="R0402" value="300"/>
+<part name="D11" library="led" deviceset="LED" device="CHIPLED_0603"/>
+<part name="GND23" library="supply1" deviceset="GND" device=""/>
 </parts>
 <sheets>
@@
 <instance part="T1" gate="G$1" x="-116.84" y="71.12" rot="R180"/>
 <instance part="J$1" gate="G$1" x="-12.7" y="60.96" rot="MR0"/>
+<instance part="R16" gate="G$1" x="152.4" y="144.78" rot="R90"/>
+<instance part="D11" gate="G$1" x="152.4" y="134.62"/>
+<instance part="GND23" gate="1" x="152.4" y="124.46"/>
 </instances>
 <busses>
@@
 <wire x1="208.28" y1="76.2" x2="236.22" y2="76.2" width="0.1524" layer="91"/>
 <label x="198.12" y="63.5" size="1.778" layer="95"/>
+</segment>
+<segment>
+<pinref part="R16" gate="G$1" pin="2"/>
+<wire x1="152.4" y1="149.86" x2="152.4" y2="154.94" width="0.1524" layer="91"/>
+<wire x1="152.4" y1="154.94" x2="157.48" y2="154.94" width="0.1524" layer="91"/>
+<label x="152.4" y="154.94" size="1.778" layer="95"/>
 </segment>
 </net>
@@
 <wire x1="-99.06" y1="-22.86" x2="-96.52" y2="-22.86" width="0.1524" layer="91"/>
 </segment>
+<segment>
+<pinref part="GND23" gate="1" pin="GND"/>
+<pinref part="D11" gate="G$1" pin="C"/>
+<wire x1="152.4" y1="127" x2="152.4" y2="129.54" width="0.1524" layer="91"/>
+</segment>
 </net>
 <net name="AREF" class="0">
@@
 </segment>
 </net>
+<net name="N$16" class="0">
+<segment>
+<pinref part="D11" gate="G$1" pin="A"/>
+<pinref part="R16" gate="G$1" pin="1"/>
+<wire x1="152.4" y1="137.16" x2="152.4" y2="139.7" width="0.1524" layer="91"/>
+</segment>
+</net>
